File: 8085basic/8085basic.kicad_pcb (KiCad board)
At the start: 2 copper layers, 163.8 x 94 mm, 46 parts, among them J1 FTDI, J2 Conn_01x11_Female, SW1 reset, SW2 SW_SPST, SW3 SW_SPDT, SW4 SW_SPST, U1 8085, U10 74LS00, U2 74LS273, U3 74LS00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

Commit message: 3/8/22
Other:
- board text added: "Margaret Black 1 / 2021 rev 2"
- board text removed: "Michael Black 1 / 2021 rev 2"
