File: arduinovideo/arduinovideo.kicad_pcb (KiCad board)
At the start: 2 copper layers, 59.7 x 49.5 mm, 8 parts, among them J1 Conn_01x12_Male, J2 Conn_01x12_Female, J3 Conn_01x16_Female, U1 ATmega328P-PU, Y1 Crystal

Commit message: 3/8/22
Other:
- board text added: "Margaret Black 1 / 2021"
- board text removed: "Michael Black 1 / 2021"
