File: risc_memory_fp/risc_memory_fp.kicad_pcb (KiCad board)
At the start: 2 copper layers, 259.1 x 149.9 mm, 110 parts, among them J1 Conn_01x03_Female, J2 Conn_01x03_Female, J3 Conn_01x08_Female, J4 Conn_01x08_Female, J5 Conn_01x08_Female, J6 Conn_01x04_Female, J7 Screw_Terminal_01x02, J8 USB_B, SW1 SW_SPDT, SW10 SW_SPDT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

Commit message: 3/8/22
Other:
- board text added: "Margaret Black 11/2020"
- board text removed: "Michael Black 11/2020"
