File: riscy_io/riscy_io.kicad_pcb (KiCad board)
At the start: 2 copper layers, 149.9 x 99.1 mm, 51 parts, among them J1 Conn_01x03_Female, J10 Conn_01x11_Female, J2 Conn_01x03_Female, J3 Conn_01x08_Female, J4 Conn_01x08_Female, J5 Conn_01x11_Female, J6 Conn_01x16_Female, J7 Conn_01x04_Female, J8 Conn_01x16_Female, J9 Conn_01x11_Female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

Commit message: 3/8/22
Other:
- board text added: "Margaret Black 1 / 2021"
- board text removed: "Michael Black 1 / 2021"
