File: riscy_pc_ir_sp/riscy_pc_ir_sp.kicad_pcb (KiCad board)
At the start: 2 copper layers, 199.4 x 149.9 mm, 138 parts, among them J1 Conn_01x03_Female, J10 Conn_01x06_Female, J11 Conn_01x08_Female, J12 Conn_01x08_Female, J2 Conn_01x03_Female, J3 Conn_01x08_Female, J4 Conn_01x08_Female, J5 Conn_01x08_Female, J6 Conn_01x08_Female, J7 Conn_01x08_Female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

Commit message: 3/8/22
Other:
- board text added: "Margaret Black 11/2020"
- board text removed: "Michael Black 11/2020"
