File: riscyalu/riscyalu.kicad_pcb (KiCad board)
At the start: 2 copper layers, 139.7 x 149.9 mm, 80 parts, among them J1 Conn_01x03_Female, J10 Conn_01x02_Female, J2 Conn_01x08_Female, J3 Conn_01x08_Female, J4 Conn_01x08_Female, J5 Conn_01x08_Female, J6 Conn_01x04_Female, J7 Conn_01x05_Female, J8 Conn_01x04_Female, J9 Conn_01x03_Female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

Commit message: 3/8/22
Other:
- board text added: "Margaret Black"
- board text removed: "Michael Black"
