File: serial/serial.kicad_pcb (KiCad board)
At the start: 2 copper layers, 199.4 x 97.8 mm, 57 parts, among them J1 FTDI, J2 rs232, J3 keyboard, J4 keyboard, J5 video, J6 baudrate, J7 USB_B, J8 video, SW1 POWER, SW2 TTLorRS232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

Commit message: 3/8/22
Other:
- board text added: "TV Typewriter Serial Board rev 2 Margaret Black 1/2021"
- board text removed: "TV Typewriter Serial Board rev 2 Michael Black 1/2021"
