File: video/video.kicad_pcb (KiCad board)
At the start: 2 copper layers, 238.8 x 99.1 mm, 72 parts, among them J1 video_out, J2 Conn_01x12_Female, Q1 2N3904, Q2 2N3904, U1 74LS161, U10 2816, U11 74LS08, U12 74LS14, U13 74LS86, U14 2016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

Commit message: 3/8/22
Other:
- board text added: "Video output rev 2 Margaret Black 1/2021"
- board text removed: "Video output rev 2 Michael Black 1/2021"
